File: kicad_project/OBD2-C.kicad_pcb (KiCad board)
At the start: 2 copper layers, 37 x 17 mm, 24 parts, among them J1 USB Type-C, J2 Conn_01x04_Socket, M1 OBDII, Q1 MMBT5551L, Q2 AO3401A

Commit message: Jumpers, pinout
Parts:
- added JP7: 1L, Jumper:SolderJumper-2_P1.3mm_Open_TrianglePad1.0x1.5mm, F.Cu at (129.6, 106.6)
- moved JP4 5.36 mm to (136.3, 106.5)
Routing:
- net GND: track 53.4 -> 42.8 mm, vias 45 -> 44
- net +12V: track 41.0 -> 35.7 mm
- net CAN1_L: track 33.5 -> 37.8 mm
- net CAN1_H: track 23.3 -> 24.0 mm
- net IGN_12V: track 40.3 -> 40.9 mm
