File: kicad_project/OBD2-C.kicad_sch (KiCad schematic)
At the start: 24 parts, among them J1 USB Type-C, J2 Conn_01x04_Socket, M1 OBDII, Q1 MMBT5551L, Q2 AO3401A

Commit message: Jumpers, pinout
Parts:
- added JP7: 1L, Jumper:SolderJumper-2_P1.3mm_Open_TrianglePad1.0x1.5mm, symbol Jumper:SolderJumper_2_Open
- J2: FT Rotation Offset (none) -> 180
Connections:
- net CAN1_L: now also JP7.2 (B)
- net at M1.10 (J1850BUS): now also JP7.1 (A)
- no-connect marks 11 -> 10
Other:
- moved on the sheet: JP2
Changed lines of the file:
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@@
 	)
 	(no_connect
-		(at 91.44 64.77)
-	)
-	(no_connect
 		(at 91.44 77.47)
 	)
@@
 	(global_label "CAN1_L"
 		(shape input)
-		(at 36.83 54.61 180)
+		(at 99.06 64.77 0)
 		(fields_autoplaced yes)
 		(effects
@@
 				(size 1.27 1.27)
 			)
-			(justify right)
+			(justify left)
 		)
 		(property "Intersheetrefs" "${INTERSHEET_REFS}"
-			(at 26.9505 54.61 0)
+			(at 108.9395 64.77 0)
 			(effects
 				(font
 					(size 1.27 1.27)
 				)
-				(justify right)
+				(justify left)
+				(hide yes)
+			)
+		)
+	)
+	(global_label "CAN1_L"
+		(shape input)
+		(at 99.06 54.61 0)
+		(fields_autoplaced yes)
+		(effects
+			(font
+				(size 1.27 1.27)
+			)
+			(justify left)
+		)
+		(property "Intersheetrefs" "${INTERSHEET_REFS}"
+			(at 108.9395 54.61 0)
+			(effects
+				(font
+					(size 1.27 1.27)
+				)
+				(justify left)
 				(hide yes)
 			)
@@
 	)
 	(symbol
+		(lib_id "Jumper:SolderJumper_2_Open")
+		(at 95.25 64.77 0)
+		(unit 1)
+		(exclude_from_sim no)
+		(in_bom no)
+		(on_board yes)
+		(dnp no)
+		(property "Reference" "JP7"
+			(at 95.25 59.436 0)
+			(effects
+				(font
+					(size 1.27 1.27)
+				)
+			)
+		)
+		(property "Value" "1L"
+			(at 95.25 61.976 0)
+			(effects
+				(font
+					(size 1.27 1.27)
+				)
+			)
+		)
+		(property "Footprint" "Jumper:SolderJumper-2_P1.3mm_Open_TrianglePad1.0x1.5mm"
+			(at 95.25 64.77 0)
+			(effects
+				(font
+					(size 1.27 1.27)
+				)
+				(hide yes)
+			)
+		)
+		(property "Datasheet" "~"
+			(at 95.25 64.77 0)
+			(effects
+				(font
+					(size 1.27 1.27)
+				)
+				(hide yes)
+			)
+		)
+		(property "Description" ""
+			(at 95.25 64.77 0)
+			(effects
+				(font
+					(size 1.27 1.27)
+				)
+				(hide yes)
+			)
+		)
+		(pin "2"
+		)
+		(pin "1"
+		)
+		(instances
+			(project "OBD2-C"
+				(path "/f2a0951e-c484-4a3e-ba5c-498011ede3e6"
+					(reference "JP7")
+					(unit 1)
+				)
+			)
+		)
+	)
+	(symbol
 		(lib_id "power:+12V")
 		(at 245.11 38.1 0)
@@
 	(symbol
 		(lib_id "Jumper:SolderJumper_2_Open")
-		(at 40.64 54.61 0)
+		(at 95.25 54.61 0)
+		(mirror y)
 		(unit 1)
 		(exclude_from_sim no)
@@
 		(dnp no)
 		(property "Reference" "JP2"
-			(at 40.64 49.276 0)
+			(at 95.25 49.276 0)
 			(effects
 				(font
@@
 		)
 		(property "Value" "GM_gnd"
-			(at 40.64 51.816 0)
+			(at 95.25 51.816 0)
 			(effects
 				(font
@@
 		)
 		(property "Footprint" "Jumper:SolderJumper-2_P1.3mm_Open_TrianglePad1.0x1.5mm"
-			(at 40.64 54.61 0)
+			(at 95.25 54.61 0)
 			(effects
 				(font
@@
 		)
 		(property "Datasheet" "~"
-			(at 40.64 54.61 0)
+			(at 95.25 54.61 0)
 			(effects
 				(font
@@
 		)
 		(property "Description" ""
-			(at 40.64 54.61 0)
+			(at 95.25 54.61 0)
 			(effects
 				(font
@@
 	(symbol
 		(lib_id "power:GND")
-		(at 44.45 54.61 90)
+		(at 91.44 54.61 270)
+		(mirror x)
 		(unit 1)
 		(exclude_from_sim no)
@@
 		(on_board yes)
 		(dnp no)
-		(fields_autoplaced yes)
 		(property "Reference" "#PWR06"
-			(at 50.8 54.61 0)
+			(at 85.09 54.61 0)
 			(effects
 				(font
@@
 		)
 		(property "Value" "GND"
-			(at 48.006 54.61 90)
+			(at 87.884 54.61 90)
 			(effects
 				(font
@@
 		)
 		(property "Footprint" ""
-			(at 44.45 54.61 0)
+			(at 91.44 54.61 0)
 			(effects
 				(font
@@
 		)
 		(property "Datasheet" ""
-			(at 44.45 54.61 0)
+			(at 91.44 54.61 0)
 			(effects
 				(font
@@
 		)
 		(property "Description" ""
-			(at 44.45 54.61 0)
+			(at 91.44 54.61 0)
 			(effects
 				(font
@@
 			(at 69.85 113.03 0)
 			(effects
+				(font
+					(size 1.27 1.27)
+				)
+				(hide yes)
+			)
+		)
+		(property "FT Rotation Offset" "180"
+			(at 69.85 113.03 0)
+			(effects
